Commit message: fixed links for xacro in .urdf files

File: src/wayfarer_description/urdf/common_properties.xacro (robot description, xacro)
@@ -1,4 +1,4 @@
 <?xml version="1.0"?>
-<robot xmlns:xacro="http://www.ros.org.wiki/xacro">
+<robot xmlns:xacro="http://www.ros.org/wiki/xacro">
     <material name="green">
         <color rgba="0.0 1.0 0.0 1.0"/>

File: src/wayfarer_description/urdf/lidar.xacro (robot description, xacro)
@@ -51,5 +51,5 @@
         <parent link="lidar_link"/>
         <child link="lidar_scan_link"/>
-        <origin xyz="0 0 0" rpy="0 0 0"/>
+        <origin xyz="0 0 0" rpy="0 0 ${pi}"/>
     </joint>
     <gazebo reference="lidar_scan_link">

File: src/wayfarer_description/urdf/mobile_base.xacro (robot description, xacro)
@@ -1,4 +1,4 @@
 <?xml version="1.0"?>
-<robot xmlns:xacro="http://www.ros.org.wiki/xacro">
+<robot xmlns:xacro="http://www.ros.org/wiki/xacro">
     <xacro:property name="scale" value="0.001"/>
     <xacro:property name="scalex" value="10"/>
@@ -75,5 +75,5 @@
         <parent link="base_footprint"/>
         <child link="base_link"/>
-        <origin xyz="0 0 ${arm_connect_height + (wheel_joint_length/2) + (wheel_radius / 2)}" rpy="0 0 ${-pi/2}"/>
+        <origin xyz="0 0 ${arm_connect_height + (wheel_joint_length/2) + (wheel_radius / 2)}" rpy="0 0 ${pi/2}"/>
     </joint>
     <joint name="top_chassis" type="fixed">

File: src/wayfarer_description/urdf/mobile_base_gazebo.xacro (robot description, xacro)
@@ -1,4 +1,4 @@
 <?xml version="1.0"?>
-<robot xmlns:xacro="http://www.ros.org.wiki/xacro">
+<robot xmlns:xacro="http://www.ros.org/wiki/xacro">
     <gazebo reference="caster_wheel_link">
         <mu1 value="0.1" />

File: src/wayfarer_description/urdf/wayfarer.urdf.xacro (robot description, xacro)
@@ -1,4 +1,4 @@
 <?xml version="1.0"?>
-<robot name="my_robot" xmlns:xacro="http://www.ros.org.wiki/xacro">
+<robot name="my_robot" xmlns:xacro="http://www.ros.org/wiki/xacro">
     <xacro:include filename="common_properties.xacro"/>
     <xacro:include filename="mobile_base.xacro"/>
