Commit message: Fixed meshes and orientations for udf

File: src/wayfarer_description/urdf/lidar.xacro (robot description, xacro)
@@ -41,15 +41,15 @@
         <parent link="top_chassis_link"/>
         <child link="lidar_link"/>
-        <origin xyz="0 0 ${-base_height+(-lidar_height/2)}" rpy=" 0 0 0"/>
+        <origin xyz="0 0 ${(base_height/2)+(lidar_height/3)}" rpy=" 0 0 0"/>
     </joint>
     <joint name="lidar_top_joint" type="fixed">
         <parent link="lidar_link"/>
         <child link="lidar_top_link"/>
-        <origin xyz="0 0 ${-lidar_height + (lidar_top_height/2)}" rpy="0 0 0"/>
+        <origin xyz="0 0 ${lidar_height/2 + (lidar_top_height/2)}" rpy="0 0 0"/>
     </joint>
     <joint name="lidar_scan_joint" type="fixed">
         <parent link="lidar_link"/>
         <child link="lidar_scan_link"/>
-        <origin xyz="0 0 0" rpy="0 0 ${pi}"/>
+        <origin xyz="0 0 0" rpy="0 0 0"/>
     </joint>
     <gazebo reference="lidar_scan_link">

File: src/wayfarer_description/urdf/mobile_base.xacro (robot description, xacro)
@@ -80,5 +80,5 @@
         <parent link="base_link"/>
         <child link="top_chassis_link"/>
-        <origin xyz="0 0 ${spacer_height + (base_height*2)}" rpy="${pi} 0 0"/>
+        <origin xyz="0 0 ${spacer_height + (base_height*2)}" rpy="0 0 0"/>
     </joint>
     <!-- Base link to arm connect links -->
@@ -86,10 +86,10 @@
         <parent link="base_link"/>
         <child link="front_arm_connect_link"/>
-        <origin xyz="0 ${base_length/4 - (arm_connect_length/2)} ${-arm_connect_height/2.0 - (base_height/2)}" rpy="${pi} 0 0"/>
+        <origin xyz="0 ${base_length/4 - (arm_connect_length/2)} ${-arm_connect_height/2.0 - (base_height/2)}" rpy="0 0 0"/>
     </joint>
     <joint name="base_back_arm_connect_joint" type="fixed">
         <parent link="base_link"/>
         <child link="back_arm_connect_link"/>
-        <origin xyz="0 ${-base_length/4 - (arm_connect_length/2)} ${-arm_connect_height/2.0 - (base_height/2)}" rpy="${pi} 0 0"/>
+        <origin xyz="0 ${-base_length/4 - (arm_connect_length/2)} ${-arm_connect_height/2.0 - (base_height/2)}" rpy="0 0 0"/>
     </joint>
     <!-- Wheel joints links -->
@@ -97,40 +97,41 @@
         <parent link="front_arm_connect_link"/>
         <child link="front_right_wheel_joint_link"/>
-        <origin xyz="${-0.51 / scalex} ${-0.09/ scalex} ${0.18/ scalex}" rpy="${-pi/2} 0 0.0"/>
+        <origin xyz="${-0.51 / scalex} ${0.45/ scalex} ${-0.18/ scalex}" rpy="0.0 0.0 0.0"/>
     </joint>
     <joint name="arm_connect_front_left_wheel_joint" type="fixed">
         <parent link="front_arm_connect_link"/>
         <child link="front_left_wheel_joint_link"/>
-        <origin xyz="${0.51/ scalex} ${-0.04/ scalex} ${0.18/ scalex}" rpy="${pi/2} ${pi} 0.0"/>
+        <origin xyz="${0.51/ scalex} ${0.40/ scalex} ${-0.18/ scalex}" rpy="0.0 0.0 ${pi}"/>
     </joint>
     <joint name="arm_connect_back_right_wheel_joint" type="fixed">
         <parent link="back_arm_connect_link"/>
         <child link="back_right_wheel_joint_link"/>
-        <origin xyz="${-0.51 / scalex} -${0.09 / scalex} ${0.18 / scalex}" rpy="${-pi/2} 0 0.0"/>
+        <origin xyz="${-0.51 / scalex} ${0.10 / scalex} ${-0.18 / scalex}" rpy="0.0 0 0.0"/>
     </joint>
     <joint name="arm_connect_back_left_wheel_joint" type="fixed">
         <parent link="back_arm_connect_link"/>
         <child link="back_left_wheel_joint_link"/>
-        <origin xyz="${0.51 / scalex} ${-0.04 / scalex} ${0.18 / scalex}" rpy="${pi/2} ${pi} 0.0"/>
+        <origin xyz="${0.51 / scalex} ${0.40 / scalex} ${-0.18 / scalex}" rpy="0.0 0.0 ${pi}"/>
     </joint>
+    <!-- Outer Wheel Joints -->
     <joint name="arm_connect_o_front_right_wheel_joint" type="fixed">
         <parent link="front_arm_connect_link"/>
         <child link="o_front_right_wheel_joint_link"/>
-        <origin xyz="${-0.51 / scalex} ${-0.45 / scalex} ${0.18 / scalex}" rpy="${pi/2} ${pi} ${pi}"/>
+        <origin xyz="${-0.51 / scalex} ${0.09 / scalex} ${-0.18 / scalex}" rpy="0 0 0"/>
     </joint>
     <joint name="arm_connect_o_back_right_wheel_joint" type="fixed">
         <parent link="back_arm_connect_link"/>
         <child link="o_back_right_wheel_joint_link"/>
-        <origin xyz="${-0.51 / scalex} ${-0.45 / scalex} ${0.18 / scalex}" rpy="${pi/2} ${pi} ${pi}"/>
+        <origin xyz="${-0.51 / scalex} ${0.45 / scalex} ${-0.18 / scalex}" rpy="0 0 0"/>
     </joint>
     <joint name="arm_connect_o_front_left_wheel_joint" type="fixed">
         <parent link="front_arm_connect_link"/>
         <child link="o_front_left_wheel_joint_link"/>
-        <origin xyz="${0.51 / scalex} ${-0.40 / scalex} ${0.18 / scalex}" rpy="${pi/2} ${pi} 0"/>
+        <origin xyz="${0.51 / scalex} ${0.04 / scalex} ${-0.18 / scalex}" rpy="${pi} ${pi} 0"/>
     </joint>
     <joint name="arm_connect_o_back_left_wheel_joint" type="fixed">
         <parent link="back_arm_connect_link"/>
         <child link="o_back_left_wheel_joint_link"/>
-        <origin xyz="${0.51 / scalex} ${-0.40 / scalex} ${0.18 / scalex}" rpy="${pi/2} ${pi} 0"/>
+        <origin xyz="${0.51 / scalex} ${0.04 / scalex} ${-0.18 / scalex}" rpy="${pi} ${pi} 0"/>
     </joint>
     <!-- Wheels -->
@@ -138,5 +139,5 @@
         <parent link="front_left_wheel_joint_link"/>
         <child link="front_r_wheel_link"/>
-        <origin xyz="${-wheel_joint_width/2 + (-wheel_length/3.5)} 0.0 ${wheel_radius /2 + (0.05 / scalex)}" rpy="0 0 ${pi/2} "/>
+        <origin xyz="${-wheel_joint_width/2 + (-wheel_length/3.5)} 0.015 ${-wheel_radius /2 + (0.05 / scalex)}" rpy="0 0 ${pi/2} "/>
         <axis xyz="0.0 -1.0 0.0"/>
     </joint>
@@ -144,5 +145,5 @@
         <parent link="front_right_wheel_joint_link"/>
         <child link="front_l_wheel_link"/>
-        <origin xyz="${-wheel_joint_width/2 + (-wheel_length/3.5)} 0.0 ${-wheel_radius /2 + (0.05 / scalex)}" rpy="0 0 ${pi/2} "/>
+        <origin xyz="${-wheel_joint_width/2 + (-wheel_length/3.5)} -0.02 ${-wheel_radius /2 + (0.05 / scalex)}" rpy="0 0 ${pi/2} "/>
         <axis xyz="0.0 1.0 0.0"/>
     </joint>
@@ -150,5 +151,5 @@
         <parent link="back_left_wheel_joint_link"/>
         <child link="back_r_wheel_link"/>
-        <origin xyz="${-wheel_joint_width/2 + (-wheel_length/3.5)} 0.0 ${wheel_radius /2 + (0.05 /scalex)}" rpy="0 0 ${pi/2} "/>
+        <origin xyz="${-wheel_joint_width/2 + (-wheel_length/3.5)} 0.015 ${-wheel_radius /2 + (0.05 /scalex)}" rpy="0 0 ${pi/2} "/>
         <axis xyz="0.0 -1.0 0.0"/>
     </joint>
@@ -156,5 +157,5 @@
         <parent link="back_right_wheel_joint_link"/>
         <child link="back_l_wheel_link"/>
-        <origin xyz="${-wheel_joint_width/2 + (-wheel_length/3.5)} 0.0 ${-wheel_radius /2 + (0.05 / scalex)}" rpy="0 0 ${pi/2} "/>
+        <origin xyz="${-wheel_joint_width/2 + (-wheel_length/3.5)} 0.015 ${-wheel_radius /2 + (0.05 / scalex)}" rpy="0 0 ${pi/2} "/>
         <axis xyz="0.0 1.0 0.0"/>
     </joint>

Commit message: fixed lidar orintaion with realtion to teh robot

File: src/wayfarer_description/urdf/lidar.xacro (robot description, xacro)
@@ -51,5 +51,5 @@
         <parent link="lidar_link"/>
         <child link="lidar_scan_link"/>
-        <origin xyz="0 0 0" rpy="0 0 0"/>
+        <origin xyz="0 0 0" rpy="0 0 ${pi/2}"/>
     </joint>
     <gazebo reference="lidar_scan_link">

File: src/wayfarer_description/urdf/mobile_base.xacro (robot description, xacro)
@@ -75,5 +75,5 @@
         <parent link="base_footprint"/>
         <child link="base_link"/>
-        <origin xyz="0 0 ${arm_connect_height + (wheel_joint_length/2) + (wheel_radius / 2)}" rpy="0 0 ${pi/2}"/>
+        <origin xyz="0 0 ${arm_connect_height + (wheel_joint_length/2) + (wheel_radius / 2)}" rpy="0 0 0"/>
     </joint>
     <joint name="top_chassis" type="fixed">
